File: batreus.kicad_pcb (KiCad board)
At the start: 2 copper layers, 237.5 x 98.8 mm, 43 parts

Commit message: export
Parts:
- added REF**: MountingHole_2.2mm_M2_ISO7380_Pad, MountingHole:MountingHole_2.2mm_M2_ISO7380_Pad, F.Cu at (66.0, 79.8)
- added REF**: MountingHole_2.2mm_M2_ISO7380_Pad, MountingHole:MountingHole_2.2mm_M2_ISO7380_Pad, F.Cu at (56.4, 115.5)
- added REF**: MountingHole_2.2mm_M2_ISO7380_Pad, MountingHole:MountingHole_2.2mm_M2_ISO7380_Pad, F.Cu at (107.6, 133.4)
- added REF**: MountingHole_2.2mm_M2_ISO7380_Pad, MountingHole:MountingHole_2.2mm_M2_ISO7380_Pad, F.Cu at (117.1, 97.6)
- added REF**: MountingHole_2.2mm_M2_ISO7380_Pad, MountingHole:MountingHole_2.2mm_M2_ISO7380_Pad, F.Cu at (191.4, 129.5)
- added REF**: MountingHole_2.2mm_M2_ISO7380_Pad, MountingHole:MountingHole_2.2mm_M2_ISO7380_Pad, F.Cu at (181.8, 93.8)
- added REF**: MountingHole_2.2mm_M2_ISO7380_Pad, MountingHole:MountingHole_2.2mm_M2_ISO7380_Pad, F.Cu at (244.6, 119.4)
- added REF**: MountingHole_2.2mm_M2_ISO7380_Pad, MountingHole:MountingHole_2.2mm_M2_ISO7380_Pad, F.Cu at (235.0, 83.7)
Routing:
- net L0: track 48.6 -> 63.0 mm
- net S1: track 367.2 -> 354.4 mm
- net R0: track 54.7 -> 66.0 mm
- net S2: track 318.9 -> 310.3 mm
- net (no net): track 478.5 -> 485.9 mm
- net S3: track 344.1 -> 337.2 mm
- net R4: track 139.4 -> 134.3 mm
- net L4: track 142.8 -> 139.4 mm
- net R5: track 155.1 -> 151.8 mm
- net R2: track 103.3 -> 100.5 mm
- net R3: track 119.7 -> 117.1 mm
- net L3: track 125.2 -> 122.7 mm
- net L5: track 158.8 -> 156.7 mm
- net R1: track 84.5 -> 85.9 mm
- net L2: track 107.8 -> 106.6 mm
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Other:
- net class Lepi added: clearance 0.24, trace_width 0.25, via_dia 0.8, via_drill 0.4

Commit message: final
Routing:
- net S0: track 350.8 -> 344.4 mm
- net S1: track 354.4 -> 348.1 mm
- net Net-(N1-Pad15): track 0.00 -> 4.16 mm
- net Net-(N1-Pad1): track 2.36 -> 0.00 mm
- net Net-(N1-Pad14): track 2.18 -> 0.00 mm
- net S2: track 310.3 -> 309.2 mm
