File: project/batreus.kicad_pcb (KiCad board)
At the start: 2 copper layers, 237.5 x 98.8 mm, 51 parts

Commit message: New case. Updated readme
Other:
- net class Default removed
- net class Lepi removed
